Commit message: fix lidar

File: src/c1_description/urdf/c1_robot.urdf (robot description, URDF)
Before this commit: robot c1_robot, 13 links, 12 joints
Joints:
- joint laser_frame_joint: origin xyz=0 0 0.02 -> xyz=0 0 0.02 rpy=0 0 3.14159

Commit message: fix localization

File: src/c1_description/urdf/c1_robot.urdf (robot description, URDF)
Before this commit: robot c1_robot, 13 links, 12 joints
Joints:
- joint laser_frame_joint: origin xyz=0 0 0.02 rpy=0 0 3.14159 -> xyz=0 0 0.02
